Commit message: UR5装在四轮差速小车上

File: robot_description/urdf/ur5.urdf (robot description, URDF)
Before this commit: robot ur5, 11 links, 10 joints
Links:
- added link caster_wheel_back, mass 1; collision cylinder length=.02 radius=0.0375; visual cylinder length=.02 radius=0.0375
- added link caster_wheel_front, mass 1; collision cylinder length=.02 radius=0.0375; visual cylinder length=.02 radius=0.0375
- added link hokuyo_link; visual box size=0.05 0.05 0.05
- added link left_back_wheel, mass 1; collision cylinder length=.02 radius=0.075; visual cylinder length=.02 radius=0.075
- added link left_front_wheel, mass 1; collision cylinder length=.02 radius=0.075; visual cylinder length=.02 radius=0.075
- added link right_back_wheel, mass 1; collision cylinder length=.02 radius=0.075; visual cylinder length=.02 radius=0.075
- added link right_front_wheel, mass 1; collision cylinder length=.02 radius=0.075; visual cylinder length=.02 radius=0.075
- added link ur5_base_link, mass 4.0; collision mesh filename=package://robot_description/meshes/ur5/collision/base.stl; visual mesh filename=package://robot_description/meshes/ur5/visual/base.dae
- link base_link: mass 4.0 -> 1; geometry collision box size=1 0.75 0.05; visual box size=1 0.75 0.05
Joints:
- added joint bottom_joint: type fixed, parent base_link, child ur5_base_link, origin xyz=0 0.15 0.1 rpy=0 0 1.57075
- added joint caster_wheel_back_joint: type fixed, parent base_link, child caster_wheel_back, origin xyz=0 -0.45 0.0375 rpy=0 -1.57075 0
- added joint caster_wheel_front_joint: type fixed, parent base_link, child caster_wheel_front, origin xyz=0 0.45 0.0375 rpy=0 -1.57075 0
- added joint hokuyo_joint: type fixed, parent base_link, child hokuyo_link, origin xyz=0 0.45 0.1 rpy=0 0 0
- added joint left_back_wheel_joint: type continuous, parent base_link, child left_back_wheel, origin xyz=-0.375 -0.45 0.075 rpy=0 -1.57075 0, axis 0 0 1, limit effort=100 velocity=100
- added joint left_front_wheel_joint: type continuous, parent base_link, child left_front_wheel, origin xyz=-0.375 0.45 0.075 rpy=0 -1.57075 0, axis 0 0 1, limit effort=100 velocity=100
- added joint right_back_wheel_joint: type continuous, parent base_link, child right_back_wheel, origin xyz=0.375 -0.45 0.075 rpy=0 -1.57075 0, axis 0 0 1, limit effort=100 velocity=100
- added joint right_front_wheel_joint: type continuous, parent base_link, child right_front_wheel, origin xyz=0.375 0.45 0.075 rpy=0 -1.57075 0, axis 0 0 1, limit effort=100 velocity=100
- joint base_link-base_fixed_joint: parent base_link -> ur5_base_link
- joint shoulder_pan_joint: parent base_link -> ur5_base_link
